Commit message: add parent argument to macro, removed world link

File: kuka_agilus_support/urdf/kr6_r900_sixx_macro.xacro (robot description, xacro)
@@ -5,8 +5,7 @@
   <xacro:include filename="$(find kuka_agilus_support)/urdf/kr_agilus_ros2_control.xacro"/>
   <xacro:include filename="$(find kuka_agilus_support)/urdf/kr_agilus_transmission.xacro"/>
-  <xacro:macro name="kuka_kr6_r900_sixx_robot" params="client_ip client_port prefix use_fake_hardware roundtrip_time *origin">
+  <xacro:macro name="kuka_kr6_r900_sixx_robot" params="client_ip client_port prefix parent:=world use_fake_hardware roundtrip_time *origin">
     <!-- ros2 control instance -->
     <xacro:kuka_agilus_ros2_control name="${prefix}kr6_r900_sixx" client_ip="${client_ip}" client_port="${client_port}" prefix="${prefix}" use_fake_hardware="${use_fake_hardware}" roundtrip_time="${roundtrip_time}"/>
-    <link name="world"/>
     <link name="${prefix}base_link">
       <visual>
@@ -117,5 +116,5 @@
     <link name="${prefix}flange"/>
     <joint name="${prefix}world-base_link" type="fixed">
-      <parent link="world"/>
+      <parent link="${parent}"/>
       <child link="${prefix}base_link"/>
       <xacro:insert_block name="origin"/>
